File: Hardware/SparkFun_Differential_I2C_Breakout_PCA9615_Qwiic.sch (EAGLE design)
At the start: 33 parts, among them J1 QWIIC_RIGHT_ANGLE, J2 QWIIC_RIGHT_ANGLE, J3 RJ45, J7 RJ45, U1 PCA9615, U2 3.3V

Commit message: updating net name to fix VDD_A issue
Connections:
- removed net VCC_1: C6.1, U2.OUT
- net VDD_A: now also C6.1, U2.OUT
Changed lines of the file:
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@@
 <pinref part="SUPPLY14" gate="G$2" pin="VCC_1"/>
+</segment>
+<segment>
+<pinref part="C6" gate="G$1" pin="1"/>
+<wire x1="66.04" y1="104.14" x2="66.04" y2="101.6" width="0.1524" layer="91"/>
+<pinref part="U2" gate="G$1" pin="OUT"/>
+<wire x1="66.04" y1="101.6" x2="66.04" y2="99.06" width="0.1524" layer="91"/>
+<wire x1="63.5" y1="101.6" x2="66.04" y2="101.6" width="0.1524" layer="91"/>
+<junction x="66.04" y="101.6"/>
+<pinref part="SUPPLY6" gate="G$2" pin="VCC_1"/>
 </segment>
 </net>
@@
 </segment>
 </net>
-<net name="VCC_1" class="0">
-<segment>
-<pinref part="C6" gate="G$1" pin="1"/>
-<wire x1="66.04" y1="104.14" x2="66.04" y2="101.6" width="0.1524" layer="91"/>
-<pinref part="U2" gate="G$1" pin="OUT"/>
-<wire x1="66.04" y1="101.6" x2="66.04" y2="99.06" width="0.1524" layer="91"/>
-<wire x1="63.5" y1="101.6" x2="66.04" y2="101.6" width="0.1524" layer="91"/>
-<junction x="66.04" y="101.6"/>
-<pinref part="SUPPLY6" gate="G$2" pin="VCC_1"/>
-</segment>
-</net>

Commit message: post design review checklist changes
Parts:
- removed JP4: JUMPER-SMT_2_NC_TRACE_SILK, SparkFun-Jumpers:JUMPER-SMT_2_NC_TRACE_SILK
- added A-B: JUMPER-SMT_2_NO_SILK, SparkFun-Jumpers:JUMPER-SMT_2_NO_SILK
- added GND\, VREG: JUMPER-SMT_2_NC_TRACE_SILK, SparkFun-Jumpers:JUMPER-SMT_2_NC_TRACE_SILK
- J1, J2: value QWIIC_RIGHT_ANGLE -> QWIIC
- renumbered JP3 to VDD_B
Connections:
- new net GRN: J3.6, J7.6
- new net N$8: U2.IN, VREG.2
- new net W_GRN: J3.3, J7.3
- net GND: now also GND\.1; no longer JP4.1
- net N$2: now also GND\.2; no longer JP4.2
- net VDD_A: now also A-B.1
- net VDD_B: now also A-B.2, VREG.1; no longer U2.IN
Other:
- note added: "Andy England"
- note added: "Based off of design by: Joel Bartlett"
- note added: "Clear the I2C jumper to remove the pullups from the bus."
- note added: "GND"
- note added: "VDD_B"
- note removed: "Cut traces on JP3 & JP4 to disconnect VDD_B and GND from cable."
- note removed: "JP2 = I2C Pullups Closed by Default"
- note removed: "Joel Bartlett"
- note removed: "Logos"
- moved on the sheet: I2C, J4, J6, J7, R7, R8
