File: Hardware/SparkFun_QwiicBus-Midpoint.sch (EAGLE design)
At the start: 33 parts, among them J1 QWIIC_RIGHT_ANGLE, J2 QWIIC_RIGHT_ANGLE, J3 RJ45, J7 RJ45, U1 PCA9615, U2 3.3V

Commit message: post design review checklist changes
Parts:
- removed J6: (no value), SparkX:I2C_STANDARD_NO_SILK
- removed JP4: JUMPER-SMT_2_NC_TRACE_SILK, SparkFun-Jumpers:JUMPER-SMT_2_NC_TRACE_SILK
- added A-B: JUMPER-SMT_2_NO_SILK, SparkFun-Jumpers:JUMPER-SMT_2_NO_SILK
- added D11: RED, SparkFun-LED:LED-RED0603
- added GND\, PWR, VREG: JUMPER-SMT_2_NC_TRACE_SILK, SparkFun-Jumpers:JUMPER-SMT_2_NC_TRACE_SILK
- added J5: (no value), SparkFun-Connectors:CONN_041X04_NO_SILK
- added R11: 1k, SparkFun-Resistors:1KOHM-0603-1/10W-1%
- J1, J2: value QWIIC_RIGHT_ANGLE -> QWIIC
- renumbered JP3 to VDD_B
Connections:
- removed net VCC_1: C6.1, U2.OUT
- new net GRN: J3.6, J7.6
- new net N$13: D11.C, R11.1
- new net N$14: PWR.2, R11.2
- new net N$8: U2.IN, VREG.2
- new net W_GRN: J3.3, J7.3
- net GND: now also GND\.1, J5.1, PWR.1; no longer J6.GND, JP4.1
- net N$2: now also GND\.2; no longer JP4.2
- net SCL: now also J5.4; no longer J6.SCL
- net SDA: now also J5.3; no longer J6.SDA
- net VDD_A: now also A-B.1, C6.1, D11.A, J5.2, U2.OUT; no longer J6.VCC
- net VDD_B: now also A-B.2, VREG.1; no longer U2.IN
Other:
- note added: "Andy England"
- note added: "Based off of design by: Joel Bartlett"
- note added: "Clear the I2C jumper to remove the pullups from the bus."
- note added: "GND"
- note added: "VDD_B"
- note removed: "Cut traces on JP3 & JP4 to disconnect VDD_B and GND from cable."
- note removed: "JP2 = I2C Pullups Closed by Default"
- note removed: "Joel Bartlett"
- note removed: "Logos"
- moved on the sheet: C1, C3, I2C, J4, J7, R7, R8

Commit message: saving all changes
Other:
- note added: "Clear the VDD_B and GND jumpers if you wan't the board to be completely disconnected from power on the RJ45 Jack. Note that if you do this, you will also need to: 1. Clear the VREG jumper 2. Close the A-B Jumper 3. Supply 3.0-5.5V to the 3.3V pin or VDDB pin"
Changed lines of the file:
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@@
 <text x="175.514" y="138.684" size="1.778" layer="95" font="vector">GND</text>
 <text x="148.844" y="7.112" size="2.54" layer="94" font="vector">Based off of design by: Joel Bartlett</text>
+<text x="101.6" y="104.14" size="1.778" layer="97" font="vector">Clear the VDD_B and GND jumpers if you wan't the board to be
+completely disconnected from power on the RJ45 Jack.
+Note that if you do this, you will also need to:
+1. Clear the VREG jumper
+2. Close the A-B Jumper
+3. Supply 3.0-5.5V to the 3.3V pin or VDDB pin</text>
 </plain>
 <instances>
@@
 </drawing>
 <compatibility>
+<note version="6.3" minversion="6.2.2" severity="warning">
+Since Version 6.2.2 text objects can contain more than one line,
+which will not be processed correctly with this version.
+</note>
 <note version="8.3" severity="warning">
 Since Version 8.3, EAGLE supports URNs for individual library

Commit message: Post checklist double check
Other:
- note added: "Cut the I2C jumper to remove the pullups from the bus."
- note added: "Cut the PWR jumper to disable the PWR LED"
- note added: "Cut the VDD_B and GND jumpers if you wan't the board to be completely disconnected from power on the RJ45 Jack. Note that if you do this, you will also need to: 1. Clear the VREG jumper 2. Close the A-B Jumper 3. Supply 3.0-5.5V to the 3.3V pin or VDDB pin"
- note removed: "Clear the I2C jumper to remove the pullups from the bus."
- note removed: "Clear the VDD_B and GND jumpers if you wan't the board to be completely disconnected from power on the RJ45 Jack. Note that if you do this, you will also need to: 1. Clear the VREG jumper 2. Close the A-B Jumper 3. Supply 3.0-5.5V to the 3.3V pin or VDDB pin"
- moved on the sheet: C1, C2, C3, C4
Changed lines of the file:
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@@
 <text x="238.76" y="7.62" size="2.54" layer="94" font="vector">v10</text>
 <wire x1="88.9" y1="81.28" x2="0" y2="81.28" width="0.2032" layer="97" style="longdash"/>
-<text x="114.3" y="76.2" size="1.778" layer="97" font="vector">Clear the I2C jumper to remove the pullups from the bus.</text>
+<text x="114.3" y="76.2" size="1.778" layer="97" font="vector">Cut the I2C jumper to remove the pullups from the bus.</text>
 <text x="2.54" y="30.48" size="2.54" layer="94" font="vector">Headers</text>
 <wire x1="88.9" y1="81.28" x2="88.9" y2="35.56" width="0.2032" layer="97" style="longdash"/>
@@
 <text x="175.514" y="138.684" size="1.778" layer="95" font="vector">GND</text>
 <text x="148.844" y="7.112" size="2.54" layer="94" font="vector">Based off of design by: Joel Bartlett</text>
-<text x="101.6" y="104.14" size="1.778" layer="97" font="vector">Clear the VDD_B and GND jumpers if you wan't the board to be
+<text x="101.6" y="104.14" size="1.778" layer="97" font="vector">Cut the VDD_B and GND jumpers if you wan't the board to be
 completely disconnected from power on the RJ45 Jack.
 Note that if you do this, you will also need to:
@@
 2. Close the A-B Jumper
 3. Supply 3.0-5.5V to the 3.3V pin or VDDB pin</text>
+<text x="12.7" y="132.08" size="1.778" layer="97" font="vector">Cut the PWR
+jumper to disable
+the PWR LED</text>
 </plain>
 <instances>
@@
 <attribute name="VALUE" x="25.4" y="152.146" size="1.778" layer="96" font="vector" align="top-center"/>
 </instance>
-<instance part="C1" gate="G$1" x="33.02" y="134.62" smashed="yes">
-<attribute name="NAME" x="34.544" y="137.541" size="1.778" layer="95" font="vector"/>
-<attribute name="VALUE" x="34.544" y="132.461" size="1.778" layer="96" font="vector"/>
-</instance>
-<instance part="C2" gate="G$1" x="60.96" y="134.62" smashed="yes">
-<attribute name="NAME" x="62.484" y="137.541" size="1.778" layer="95" font="vector"/>
-<attribute name="VALUE" x="62.484" y="132.461" size="1.778" layer="96" font="vector"/>
-</instance>
-<instance part="C3" gate="G$1" x="45.72" y="134.62" smashed="yes">
-<attribute name="NAME" x="47.244" y="137.541" size="1.778" layer="95" font="vector"/>
-<attribute name="VALUE" x="47.244" y="132.461" size="1.778" layer="96" font="vector"/>
-</instance>
-<instance part="C4" gate="G$1" x="73.66" y="134.62" smashed="yes">
-<attribute name="NAME" x="75.184" y="137.541" size="1.778" layer="95" font="vector"/>
-<attribute name="VALUE" x="75.184" y="132.461" size="1.778" layer="96" font="vector"/>
-</instance>
-<instance part="GND6" gate="1" x="33.02" y="127" smashed="yes">
-<attribute name="VALUE" x="33.02" y="126.746" size="1.778" layer="96" font="vector" align="top-center"/>
-</instance>
-<instance part="GND7" gate="1" x="45.72" y="127" smashed="yes">
-<attribute name="VALUE" x="45.72" y="126.746" size="1.778" layer="96" font="vector" align="top-center"/>
-</instance>
-<instance part="GND8" gate="1" x="60.96" y="127" smashed="yes">
-<attribute name="VALUE" x="60.96" y="126.746" size="1.778" layer="96" font="vector" align="top-center"/>
-</instance>
-<instance part="GND9" gate="1" x="73.66" y="127" smashed="yes">
-<attribute name="VALUE" x="73.66" y="126.746" size="1.778" layer="96" font="vector" align="top-center"/>
-</instance>
-<instance part="SUPPLY7" gate="G$2" x="33.02" y="142.24" smashed="yes">
-<attribute name="VALUE" x="33.02" y="145.034" size="1.778" layer="96" font="vector" align="bottom-center"/>
-</instance>
-<instance part="SUPPLY8" gate="G$2" x="45.72" y="142.24" smashed="yes">
-<attribute name="VALUE" x="45.72" y="145.034" size="1.778" layer="96" font="vector" align="bottom-center"/>
-</instance>
-<instance part="SUPPLY9" gate="G$1" x="60.96" y="142.24" smashed="yes">
-<attribute name="VALUE" x="60.96" y="145.034" size="1.778" layer="96" font="vector" align="bottom-center"/>
-</instance>
-<instance part="SUPPLY10" gate="G$1" x="73.66" y="142.24" smashed="yes">
-<attribute name="VALUE" x="73.66" y="145.034" size="1.778" layer="96" font="vector" align="bottom-center"/>
+<instance part="C1" gate="G$1" x="40.64" y="134.62" smashed="yes">
+<attribute name="NAME" x="42.164" y="137.541" size="1.778" layer="95" font="vector"/>
+<attribute name="VALUE" x="42.164" y="132.461" size="1.778" layer="96" font="vector"/>
+</instance>
+<instance part="C2" gate="G$1" x="66.04" y="134.62" smashed="yes">
+<attribute name="NAME" x="67.564" y="137.541" size="1.778" layer="95" font="vector"/>
+<attribute name="VALUE" x="67.564" y="132.461" size="1.778" layer="96" font="vector"/>
+</instance>
+<instance part="C3" gate="G$1" x="53.34" y="134.62" smashed="yes">
+<attribute name="NAME" x="54.864" y="137.541" size="1.778" layer="95" font="vector"/>
+<attribute name="VALUE" x="54.864" y="132.461" size="1.778" layer="96" font="vector"/>
+</instance>
+<instance part="C4" gate="G$1" x="78.74" y="134.62" smashed="yes">
+<attribute name="NAME" x="80.264" y="137.541" size="1.778" layer="95" font="vector"/>
+<attribute name="VALUE" x="80.264" y="132.461" size="1.778" layer="96" font="vector"/>
+</instance>
+<instance part="GND6" gate="1" x="40.64" y="127" smashed="yes">
+<attribute name="VALUE" x="40.64" y="126.746" size="1.778" layer="96" font="vector" align="top-center"/>
+</instance>
+<instance part="GND7" gate="1" x="53.34" y="127" smashed="yes">
+<attribute name="VALUE" x="53.34" y="126.746" size="1.778" layer="96" font="vector" align="top-center"/>
+</instance>
+<instance part="GND8" gate="1" x="66.04" y="127" smashed="yes">
+<attribute name="VALUE" x="66.04" y="126.746" size="1.778" layer="96" font="vector" align="top-center"/>
+</instance>
+<instance part="GND9" gate="1" x="78.74" y="127" smashed="yes">
+<attribute name="VALUE" x="78.74" y="126.746" size="1.778" layer="96" font="vector" align="top-center"/>
+</instance>
+<instance part="SUPPLY7" gate="G$2" x="40.64" y="142.24" smashed="yes">
+<attribute name="VALUE" x="40.64" y="145.034" size="1.778" layer="96" font="vector" align="bottom-center"/>
+</instance>
+<instance part="SUPPLY8" gate="G$2" x="53.34" y="142.24" smashed="yes">
+<attribute name="VALUE" x="53.34" y="145.034" size="1.778" layer="96" font="vector" align="bottom-center"/>
+</instance>
+<instance part="SUPPLY9" gate="G$1" x="66.04" y="142.24" smashed="yes">
+<attribute name="VALUE" x="66.04" y="145.034" size="1.778" layer="96" font="vector" align="bottom-center"/>
+</instance>
+<instance part="SUPPLY10" gate="G$1" x="78.74" y="142.24" smashed="yes">
+<attribute name="VALUE" x="78.74" y="145.034" size="1.778" layer="96" font="vector" align="bottom-center"/>
 </instance>
 <instance part="J3" gate="JP1" x="152.4" y="144.78" smashed="yes">
@@
 <pinref part="C1" gate="G$1" pin="2"/>
 <pinref part="GND6" gate="1" pin="GND"/>
-<wire x1="33.02" y1="129.54" x2="33.02" y2="132.08" width="0.1524" layer="91"/>
+<wire x1="40.64" y1="129.54" x2="40.64" y2="132.08" width="0.1524" layer="91"/>
 </segment>
 <segment>
 <pinref part="C3" gate="G$1" pin="2"/>
 <pinref part="GND7" gate="1" pin="GND"/>
-<wire x1="45.72" y1="129.54" x2="45.72" y2="132.08" width="0.1524" layer="91"/>
+<wire x1="53.34" y1="129.54" x2="53.34" y2="132.08" width="0.1524" layer="91"/>
 </segment>
 <segment>
 <pinref part="C2" gate="G$1" pin="2"/>
 <pinref part="GND8" gate="1" pin="GND"/>
-<wire x1="60.96" y1="129.54" x2="60.96" y2="132.08" width="0.1524" layer="91"/>
+<wire x1="66.04" y1="129.54" x2="66.04" y2="132.08" width="0.1524" layer="91"/>
 </segment>
 <segment>
 <pinref part="C4" gate="G$1" pin="2"/>
 <pinref part="GND9" gate="1" pin="GND"/>
-<wire x1="73.66" y1="129.54" x2="73.66" y2="132.08" width="0.1524" layer="91"/>
+<wire x1="78.74" y1="129.54" x2="78.74" y2="132.08" width="0.1524" layer="91"/>
 </segment>
 <segment>
@@
 <pinref part="C1" gate="G$1" pin="1"/>
 <pinref part="SUPPLY7" gate="G$2" pin="VCC_1"/>
-<wire x1="33.02" y1="142.24" x2="33.02" y2="139.7" width="0.1524" layer="91"/>
+<wire x1="40.64" y1="142.24" x2="40.64" y2="139.7" width="0.1524" layer="91"/>
 </segment>
 <segment>
 <pinref part="C3" gate="G$1" pin="1"/>
 <pinref part="SUPPLY8" gate="G$2" pin="VCC_1"/>
-<wire x1="45.72" y1="142.24" x2="45.72" y2="139.7" width="0.1524" layer="91"/>
+<wire x1="53.34" y1="142.24" x2="53.34" y2="139.7" width="0.1524" layer="91"/>
 </segment>
 <segment>
@@
 <pinref part="C2" gate="G$1" pin="1"/>
 <pinref part="SUPPLY9" gate="G$1" pin="VCC_2"/>
-<wire x1="60.96" y1="142.24" x2="60.96" y2="139.7" width="0.1524" layer="91"/>
+<wire x1="66.04" y1="142.24" x2="66.04" y2="139.7" width="0.1524" layer="91"/>
 </segment>
 <segment>
 <pinref part="C4" gate="G$1" pin="1"/>
 <pinref part="SUPPLY10" gate="G$1" pin="VCC_2"/>
-<wire x1="73.66" y1="142.24" x2="73.66" y2="139.7" width="0.1524" layer="91"/>
-</segment>
-<segment>
+<wire x1="78.74" y1="142.24" x2="78.74" y2="139.7" width="0.1524" layer="91"/>
+</segment>
+<segment>
