File: Hardware/SparkFun_QwiicBus-Midpoint.sch (EAGLE design)
At the start: 64 parts, among them J1 QWIIC, J2 QWIIC, J3 RJ45, J7 RJ45, Q1 SI7120AD, U1 PCA9615, U3 LMR33630, U4 LTC4231 Hot Swap Controller

Commit message: pushing unsaved changes from double check
Other:
- note added: "Delays start-up for 40 ms"
- note added: "Hot Swap Controller"
- note added: "v14"
- note removed: "VIN: 3.8V-32V"
- note removed: "v13"
Changed lines of the file:
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@@
 <wire x1="88.9" y1="114.3" x2="0" y2="114.3" width="0.2032" layer="97" style="longdash"/>
 <wire x1="88.9" y1="185.42" x2="88.9" y2="119.38" width="0.2032" layer="97" style="longdash"/>
-<text x="238.76" y="7.62" size="2.54" layer="94" font="vector">v13</text>
+<text x="238.76" y="7.62" size="2.54" layer="94" font="vector">v14</text>
 <wire x1="88.9" y1="119.38" x2="88.9" y2="114.3" width="0.2032" layer="97" style="longdash"/>
 <wire x1="73.66" y1="71.12" x2="0" y2="71.12" width="0.2032" layer="97" style="longdash"/>
@@
 the PWR LED</text>
 <text x="78.74" y="91.44" size="2.54" layer="94" font="vector">3.8-36V In, 3.3V 3A Out Buck Regulator</text>
-<text x="78.74" y="88.9" size="1.27" layer="94" font="vector">VIN: 3.8V-32V</text>
 <text x="91.44" y="99.06" size="1.27" layer="97" font="vector">Depending on load and distance requirements, there are several different ways to power the Midpoint/Endpoint combo.
 ---
@@
 <plain>
 <text x="166.116" y="11.176" size="2.54" layer="94" font="vector">Andy England</text>
-<text x="238.76" y="7.62" size="2.54" layer="94" font="vector">v13</text>
+<text x="238.76" y="7.62" size="2.54" layer="94" font="vector">v14</text>
 <text x="148.844" y="7.112" size="2.54" layer="94" font="vector">Based off of design by: Joel Bartlett</text>
+<text x="2.54" y="180.34" size="2.54" layer="94" font="vector">Hot Swap Controller</text>
+<text x="2.54" y="177.8" size="1.778" layer="94" font="vector">Delays start-up for 40 ms</text>
 </plain>
 <instances>

Commit message: rolling back to non hot swap version
Parts:
- removed C13: 20nF, hotswap:20NF-0603-50V-10%
- removed C17: 39nF, hotswap:39NF-0805-50V-10%
- removed D1: SMAJ36A, hotswap:DIODE_TVS_UNI
- removed FRAME2: FRAME-LETTER, SparkFun-Aesthetics:FRAME-LETTER
- removed Q1: SI7120AD, hotswap:SI7120AD
- removed R10: 23m, hotswap:23MILLIOHM
- removed R12: 10, SparkFun-Resistors:10OHM-0603-1/10W-1%
- removed R13: 1k, SparkFun-Resistors:1KOHM-0603-1/10W-1%
- removed R14: 20k, SparkFun-Resistors:20KOHM-0603-1/10W-1%
- removed R15: 1M, SparkFun-Resistors:1MOHM-0603-1/4W-5%
- removed R4: 1.65K, hotswap:1.65KOHM
- removed R5: 32.4k, hotswap:32.4KOHM
- removed R6: 4.22k, hotswap:4.22KOHM
- removed R9: 1020K, hotswap:1020KOHM
- removed U4: LTC4231 Hot Swap Controller, hotswap:LTC4231
Connections:
- removed net N$10: R4.2, R9.1, U4.UVL
- removed net N$11: Q1.G, R12.2
- removed net N$12: Q1.D, R10.2, U4.SENSE
- removed net N$16: R12.1, R13.2, U4.GATE
- removed net N$17: C13.1, R13.1
- removed net N$19: R14.1, U4.STATUS
- removed net N$2: R5.1, U4.GNDSW
- removed net N$20: R15.1, U4.!SHDN
- removed net N$21: C17.1, U4.TIMER
- removed net N$5: R5.2, R6.1, U4.OV
- removed net N$8: R4.1, R6.2, U4.UVH
- removed net PWR_SRC: D1.C, PSEL.2, R10.1, R15.2, R9.2, U4.IN
- net GND: no longer C13.2, C17.2, D1.A, U4.GND
- net VREG_IN: now also PSEL.2; no longer Q1.S, R14.2, U4.SOURCE
Other:
- note added: "VIN: 3.8V-32V"
- note added: "v13"
- note removed: "Delays start-up for 40 ms"
- note removed: "Hot Swap Controller"
- note removed: "v14"
