File: Hardware/SparkFun_QwiicBus-Midpoint.brd (EAGLE design)
At the start: 48.3 x 27.9 mm, 60 parts, among them J1 QWIIC, J2 QWIIC, J3 RJ45, J7 RJ45, U1 PCA9615, U2 AP63203

Commit message: Sprinkling in some vias
Routing:
- net GND: vias 11 -> 29
Changed lines of the file:
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@@
 <wire x1="21.871" y1="12.9825" x2="22.9585" y2="12.9825" width="0.2032" layer="1"/>
 <wire x1="22.9585" y1="12.9825" x2="23.114" y2="12.827" width="0.2032" layer="1"/>
+<via x="13.462" y="18.923" extent="1-16" drill="0.381"/>
+<via x="13.716" y="17.272" extent="1-16" drill="0.381"/>
+<via x="14.478" y="18.288" extent="1-16" drill="0.381"/>
+<via x="15.621" y="19.05" extent="1-16" drill="0.381"/>
+<via x="18.796" y="19.431" extent="1-16" drill="0.381"/>
+<via x="15.113" y="9.779" extent="1-16" drill="0.381"/>
+<via x="14.478" y="13.589" extent="1-16" drill="0.381"/>
+<via x="17.399" y="19.304" extent="1-16" drill="0.381"/>
+<via x="20.066" y="22.098" extent="1-16" drill="0.381"/>
+<via x="7.366" y="24.511" extent="1-16" drill="0.381"/>
+<via x="8.128" y="25.273" extent="1-16" drill="0.381"/>
+<via x="2.54" y="20.828" extent="1-16" drill="0.381"/>
+<via x="26.67" y="22.86" extent="1-16" drill="0.381"/>
+<via x="6.223" y="12.7" extent="1-16" drill="0.381"/>
+<via x="6.35" y="17.78" extent="1-16" drill="0.381"/>
+<via x="5.969" y="10.287" extent="1-16" drill="0.381"/>
+<via x="3.81" y="10.16" extent="1-16" drill="0.381"/>
+<via x="5.08" y="6.223" extent="1-16" drill="0.381"/>
 </signal>
 <signal name="VDD_B">

Commit message: post review changes
Parts:
- removed H1: STAND-OFF, SparkFun-Hardware:STAND-OFF
- added U$11, U$14: (no value), output:#VDDA##0
- added U$16, U$5: (no value), output:#HV##0
- added U$17: (no value), output:NC0
- added U$18: (no value), output:HV0
- added U$19: (no value), output:VDDA0
- added U$20: (no value), SparkFun-Aesthetics:ORDERING_INSTRUCTIONS
- renumbered HV to HV_IN, HVGND to HV_GND, VDD_B to VDD_A
Connections:
- net VDD_B renamed VDD_A
Other:
- board text added: "2 Oz Copper"
Changed lines of the file:
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@@
 <text x="10.16" y="40.64" size="1.778" layer="47" font="vector">Units in Inches</text>
 <dimension x1="2.54" y1="3.81" x2="0" y2="3.81" x3="1.27" y3="-3.81" textsize="1.778" layer="47" unit="inch"/>
+<text x="54.61" y="31.75" size="1.778" layer="51" font="vector">2 Oz Copper</text>
 </plain>
 <attributes>
@@
 <attribute name="VALUE" x="24.13" y="11.938" size="0.6096" layer="27" font="vector" ratio="20" rot="R180" align="top-center"/>
 </element>
-<element name="H1" library="SparkFun-Hardware" package="STAND-OFF" value="STAND-OFF" x="-21.59" y="0" smashed="yes" rot="R90">
-<attribute name="NAME" x="-23.622" y="0" size="0.6096" layer="25" font="vector" ratio="20" rot="R90" align="bottom-center"/>
-<attribute name="VALUE" x="-19.558" y="0" size="0.6096" layer="27" font="vector" ratio="20" rot="R90" align="top-center"/>
-</element>
 <element name="H2" library="SparkFun-Hardware" package="STAND-OFF" value="STAND-OFF" x="22.86" y="24.13" smashed="yes" rot="R90">
 <attribute name="NAME" x="20.828" y="24.13" size="0.6096" layer="25" font="vector" ratio="20" rot="R90" align="bottom-center"/>
@@
 </element>
 <element name="LOGO1" library="SparkFun-Aesthetics" package="OSHW-LOGO-M" value="OSHW-LOGOM" x="12.7" y="3.81" smashed="yes" rot="MR0"/>
-<element name="VDD_B" library="SparkFun-Jumpers" package="SMT-JUMPER_2_NC_TRACE_SILK" package3d_urn="urn:adsk.eagle:package:39281/1" value="JUMPER-SMT_2_NC_TRACE_SILK" x="39.37" y="6.35" smashed="yes" rot="MR0">
+<element name="VDD_A" library="SparkFun-Jumpers" package="SMT-JUMPER_2_NC_TRACE_SILK" package3d_urn="urn:adsk.eagle:package:39281/1" value="JUMPER-SMT_2_NC_TRACE_SILK" x="39.37" y="6.35" smashed="yes" rot="MR0">
 <attribute name="NAME" x="39.37" y="7.493" size="0.6096" layer="26" font="vector" ratio="20" rot="MR0" align="bottom-center"/>
 <attribute name="VALUE" x="39.37" y="5.207" size="0.6096" layer="28" font="vector" ratio="20" rot="MR0" align="top-center"/>
@@
 <attribute name="VALUE" x="22.2885" y="1.651" size="0.6096" layer="27" font="vector" ratio="20" align="top-center"/>
 </element>
-<element name="HVGND" library="SparkFun-Jumpers" package="SMT-JUMPER_2_NC_TRACE_SILK" package3d_urn="urn:adsk.eagle:package:39281/1" value="JUMPER-SMT_2_NC_TRACE_SILK" x="34.29" y="21.59" smashed="yes" rot="MR180">
+<element name="HV_GND" library="SparkFun-Jumpers" package="SMT-JUMPER_2_NC_TRACE_SILK" package3d_urn="urn:adsk.eagle:package:39281/1" value="JUMPER-SMT_2_NC_TRACE_SILK" x="34.29" y="21.59" smashed="yes" rot="MR180">
 <attribute name="NAME" x="34.29" y="20.447" size="0.6096" layer="26" font="vector" ratio="20" rot="MR180" align="bottom-center"/>
 <attribute name="VALUE" x="34.29" y="22.733" size="0.6096" layer="28" font="vector" ratio="20" rot="MR180" align="top-center"/>
 </element>
-<element name="HV" library="SparkFun-Jumpers" package="SMT-JUMPER_2_NC_TRACE_SILK" package3d_urn="urn:adsk.eagle:package:39281/1" value="JUMPER-SMT_2_NC_TRACE_SILK" x="34.29" y="6.35" smashed="yes" rot="MR0">
+<element name="HV_IN" library="SparkFun-Jumpers" package="SMT-JUMPER_2_NC_TRACE_SILK" package3d_urn="urn:adsk.eagle:package:39281/1" value="JUMPER-SMT_2_NC_TRACE_SILK" x="34.29" y="6.35" smashed="yes" rot="MR0">
 <attribute name="NAME" x="34.29" y="7.493" size="0.6096" layer="26" font="vector" ratio="20" rot="MR0" align="bottom-center"/>
 <attribute name="VALUE" x="34.29" y="5.207" size="0.6096" layer="28" font="vector" ratio="20" rot="MR0" align="top-center"/>
@@
 <attribute name="VALUE" x="0" y="7.112" size="0.6096" layer="27" font="vector" ratio="20"/>
 </element>
+<element name="U$11" library="output" package="#VDDA##0" value="" x="39.37" y="5.588" smashed="yes" rot="MR270"/>
+<element name="U$14" library="output" package="#VDDA##0" value="" x="36.83" y="5.588" smashed="yes" rot="MR270"/>
+<element name="U$5" library="output" package="#HV##0" value="" x="34.29" y="22.352" smashed="yes" rot="MR90"/>
+<element name="U$16" library="output" package="#HV##0" value="" x="34.29" y="5.588" smashed="yes" rot="MR270"/>
+<element name="U$18" library="output" package="HV0" value="" x="22.352" y="5.207" smashed="yes" rot="R90"/>
+<element name="U$19" library="output" package="VDDA0" value="" x="19.304" y="5.207" smashed="yes" rot="R90"/>
+<element name="U$17" library="output" package="NC0" value="" x="25.273" y="5.207" smashed="yes" rot="R90"/>
+<element name="U$20" library="SparkFun-Aesthetics" package="ORDERING_INSTRUCTIONS" value="" x="53.34" y="43.18" smashed="yes"/>
 </elements>
 <signals>
@@
 <contactref element="C6" pad="2"/>
 <contactref element="C7" pad="2"/>
-<contactref element="HVGND" pad="1"/>
+<contactref element="HV_GND" pad="1"/>
 <polygon width="0.254" layer="1" thermals="no">
 <vertex x="12.6365" y="12.7635"/>
@@
 <via x="5.08" y="6.223" extent="1-16" drill="0.381"/>
 </signal>
-<signal name="VDD_B">
-<contactref element="VDD_B" pad="1"/>
+<signal name="VDD_A">
+<contactref element="VDD_A" pad="1"/>
 <contactref element="S1" pad="1"/>
 <wire x1="19.2885" y1="4.925" x2="19.2885" y2="6.2333" width="0.7112" layer="1"/>
@@
 <contactref element="J7" pad="5"/>
 <contactref element="J3" pad="5"/>
-<contactref element="VDD_B" pad="2"/>
+<contactref element="VDD_A" pad="2"/>
 <wire x1="37.4523" y1="9.4107" x2="37.4523" y2="12.3795125" width="0.2032" layer="16"/>
 <wire x1="37.465" y1="9.398" x2="37.4523" y2="9.4107" width="0.2032" layer="16"/>
@@
 <wire x1="44.069" y1="15.621" x2="44.069" y2="18.034" width="0.2032" layer="1"/>
 <wire x1="34.925" y1="9.398" x2="34.925" y2="9.3882875" width="0.2032" layer="1"/>
-<contactref element="HV" pad="1"/>
+<contactref element="HV_IN" pad="1"/>
 <wire x1="34.925" y1="7.7343" x2="34.8107" y2="7.62" width="0.3048" layer="16"/>
 <wire x1="34.8107" y1="7.62" x2="34.8107" y2="6.35" width="0.3048" layer="16"/>
@@
 <wire x1="37.4594875" y1="18.863709375" x2="37.4594875" y2="17.0997125" width="0.2032" layer="1"/>
 <wire x1="38.735" y1="11.938" x2="38.7858" y2="11.8872" width="0.2032" layer="1"/>
-<contactref element="HVGND" pad="2"/>
+<contactref element="HV_GND" pad="2"/>
 <wire x1="34.925" y1="19.3772125" x2="34.925" y2="15.875" width="0.3048" layer="16"/>
 <wire x1="34.925" y1="19.3772125" x2="34.8107" y2="19.4915125" width="0.3048" layer="16"/>
@@
 <contactref element="U2" pad="2"/>
 <contactref element="C8" pad="2"/>
-<contactref element="HV" pad="2"/>
+<contactref element="HV_IN" pad="2"/>
 <polygon width="0.254" layer="1" thermals="no">
 <vertex x="15.3035" y="12.7635"/>

Commit message: ordering protos
Parts:
- HV_GND, HV_IN: value JUMPER-SMT_2_NC_TRACE_SILK -> JUMPER-SMT_2_NO_SILK; device SparkFun-Jumpers:SMT-JUMPER_2_NC_TRACE_SILK -> SparkFun-Jumpers:SMT-JUMPER_2_NO_SILK
Changed lines of the file:
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@@
 <element name="C6" library="SparkFun-Capacitors" package="1206" value="22uF" x="10.287" y="18.415" smashed="yes">
 <attribute name="NAME" x="10.287" y="19.177" size="0.6096" layer="25" font="vector" ratio="20" align="bottom-center"/>
-<attribute name="PROD_ID" value="CAP-17073" x="5.207" y="22.225" size="1.778" layer="27" display="off"/>
+<attribute name="PROD_ID" value="CAP-15263" x="5.207" y="22.225" size="1.778" layer="27" display="off"/>
 <attribute name="VALUE" x="10.287" y="17.653" size="0.6096" layer="27" font="vector" ratio="20" align="top-center"/>
 </element>
 <element name="C7" library="SparkFun-Capacitors" package="1206" value="22uF" x="10.287" y="15.875" smashed="yes">
 <attribute name="NAME" x="10.287" y="16.637" size="0.6096" layer="25" font="vector" ratio="20" align="bottom-center"/>
-<attribute name="PROD_ID" value="CAP-17073" x="1.397" y="15.875" size="1.778" layer="27" display="off"/>
+<attribute name="PROD_ID" value="CAP-15263" x="1.397" y="15.875" size="1.778" layer="27" display="off"/>
 <attribute name="VALUE" x="10.287" y="15.113" size="0.6096" layer="27" font="vector" ratio="20" align="top-center"/>
 </element>
@@
 <attribute name="VALUE" x="22.2885" y="1.651" size="0.6096" layer="27" font="vector" ratio="20" align="top-center"/>
 </element>
-<element name="HV_GND" library="SparkFun-Jumpers" package="SMT-JUMPER_2_NC_TRACE_SILK" package3d_urn="urn:adsk.eagle:package:39281/1" value="JUMPER-SMT_2_NC_TRACE_SILK" x="34.29" y="21.59" smashed="yes" rot="MR180">
+<element name="HV_GND" library="SparkFun-Jumpers" package="SMT-JUMPER_2_NO_SILK" package3d_urn="urn:adsk.eagle:package:39279/1" value="JUMPER-SMT_2_NO_SILK" x="34.29" y="21.59" smashed="yes" rot="MR180">
 <attribute name="NAME" x="34.29" y="20.447" size="0.6096" layer="26" font="vector" ratio="20" rot="MR180" align="bottom-center"/>
 <attribute name="VALUE" x="34.29" y="22.733" size="0.6096" layer="28" font="vector" ratio="20" rot="MR180" align="top-center"/>
 </element>
-<element name="HV_IN" library="SparkFun-Jumpers" package="SMT-JUMPER_2_NC_TRACE_SILK" package3d_urn="urn:adsk.eagle:package:39281/1" value="JUMPER-SMT_2_NC_TRACE_SILK" x="34.29" y="6.35" smashed="yes" rot="MR0">
+<element name="HV_IN" library="SparkFun-Jumpers" package="SMT-JUMPER_2_NO_SILK" package3d_urn="urn:adsk.eagle:package:39279/1" value="JUMPER-SMT_2_NO_SILK" x="34.29" y="6.35" smashed="yes" rot="MR0">
 <attribute name="NAME" x="34.29" y="7.493" size="0.6096" layer="26" font="vector" ratio="20" rot="MR0" align="bottom-center"/>
 <attribute name="VALUE" x="34.29" y="5.207" size="0.6096" layer="28" font="vector" ratio="20" rot="MR0" align="top-center"/>
@@
 <wire x1="34.925" y1="9.398" x2="34.925" y2="9.3882875" width="0.2032" layer="1"/>
 <contactref element="HV_IN" pad="1"/>
-<wire x1="34.925" y1="7.7343" x2="34.8107" y2="7.62" width="0.3048" layer="16"/>
-<wire x1="34.8107" y1="7.62" x2="34.8107" y2="6.35" width="0.3048" layer="16"/>
 <wire x1="34.925" y1="9.398" x2="34.925" y2="7.7343" width="0.3048" layer="16"/>
+<wire x1="34.6964" y1="7.5057" x2="34.6964" y2="6.35" width="0.3048" layer="16"/>
+<wire x1="34.925" y1="7.7343" x2="34.6964" y2="7.5057" width="0.3048" layer="16"/>
 </signal>
 <signal name="GRN_N">
@@
 <wire x1="38.735" y1="11.938" x2="38.7858" y2="11.8872" width="0.2032" layer="1"/>
 <contactref element="HV_GND" pad="2"/>
-<wire x1="34.925" y1="19.3772125" x2="34.925" y2="15.875" width="0.3048" layer="16"/>
-<wire x1="34.925" y1="19.3772125" x2="34.8107" y2="19.4915125" width="0.3048" layer="16"/>
-<wire x1="34.8107" y1="21.59" x2="34.8107" y2="19.4915125" width="0.3048" layer="16"/>
+<wire x1="34.925" y1="15.875" x2="34.925" y2="19.3772125" width="0.3048" layer="16"/>
+<wire x1="34.6964" y1="19.6058125" x2="34.6964" y2="21.59" width="0.3048" layer="16"/>
+<wire x1="34.925" y1="19.3772125" x2="34.6964" y2="19.6058125" width="0.3048" layer="16"/>
 </signal>
 <signal name="N$7">
@@
 <wire x1="17.526" y1="12.065" x2="17.78" y2="12.319" width="0.2032" layer="1"/>
 <wire x1="17.78" y1="12.319" x2="17.78" y2="13.97" width="0.2032" layer="1"/>
-<wire x1="33.7693" y1="6.35" x2="32.512" y2="6.35" width="0.3048" layer="16"/>
+<wire x1="33.8836" y1="6.35" x2="32.512" y2="6.35" width="0.3048" layer="16"/>
 <via x="20.574" y="15.621" extent="1-16" drill="0.381"/>
 <wire x1="20.574" y1="15.621" x2="17.526" y2="15.621" width="1.27" layer="1"/>
-<wire x1="17.526" y1="15.621" x2="17.399" y2="15.748" width="0.7112" layer="1"/>
 <wire x1="23.241" y1="15.621" x2="20.574" y2="15.621" width="0.3048" layer="16"/>
 <wire x1="32.512" y1="6.35" x2="23.241" y2="15.621" width="0.3048" layer="16"/>

Commit message: post FarmHand Review
Parts:
- removed HV_IN: JUMPER-SMT_2_NO_SILK, SparkFun-Jumpers:SMT-JUMPER_2_NO_SILK
- removed L1: 4.7μH, SparkFun-Coils:INDUCTOR_4X4MM
- removed S1: (no value), SparkFun-Switches:SWITCH_SP3T_SMD
- removed U$25: (no value), output:#GRN#0
- removed U$26, U$27: (no value), output:#GRN#W#0
- removed U$5: (no value), output:#HV##0
- removed U2: AP63203, SparkFun-IC-Power:SOT23-6
- removed VDD_A: JUMPER-SMT_2_NC_TRACE_SILK, SparkFun-Jumpers:SMT-JUMPER_2_NC_TRACE_SILK
- added BUCK_BP: JUMPER-SMT_2_NC_TRACE_SILK, SparkFun-Jumpers:SMT-JUMPER_2_NC_TRACE_SILK
- added C10, C11: 22UF, SparkFun-Capacitors:1210
- added C12: 100uF, SparkFun-Capacitors:8X10.5
- added C14, C9: 0.1uF, SparkFun-Capacitors:0603
- added C15: 0.22uF, SparkFun-Capacitors:0603
- added L2: 4.7μH, SparkFun-Coils:INDUCTOR_4X4MM
- added PSEL: JUMPER-SMT_3_NO_SILK, SparkFun-Jumpers:SMT-JUMPER_3_NO_SILK
- added R1, R3: 100k, SparkFun-Resistors:0603
- added R2: 43k, SparkFun-Resistors:0603
- added TP1: TEST-POINT3, SparkFun-Connectors:PAD.03X.03
- added U3: LMR33630, SparkFun-IC-Power:VQFN-HR-12
- C5: value 0.1uF -> 1.0uF
- C6, C7: value 22uF -> 4.7uF; device SparkFun-Capacitors:1206 -> SparkFun-Capacitors:0805
- C8: value 10uF -> 0.22uF; device SparkFun-Capacitors:1210 -> SparkFun-Capacitors:0603
- HV_GND: value JUMPER-SMT_2_NO_SILK -> JUMPER-SMT_2_NC_TRACE_SILK; device SparkFun-Jumpers:SMT-JUMPER_2_NO_SILK -> SparkFun-Jumpers:SMT-JUMPER_2_NC_TRACE_SILK
- U$11: device output:#VDDA##0 -> output:#GND2#0
- U$14: device output:#VDDA##0 -> output:#GND1#0
- U$16: device output:#HV##0 -> output:#VCC2#0
- U$17: device output:NC0 -> output:#PSEL#0
- U$18: device output:HV0 -> output:10
- U$19: device output:VDDA0 -> output:20
- U$24: device output:#GRN#0 -> output:#GND2#0
- moved U$24 27.0 mm to (21.6, 24.9), flipped to the bottom, turned to 270 degrees
- moved J6 26.2 mm to (24.1, 25.4), turned to 180 degrees
- moved U$16 21.8 mm to (24.1, 24.8)
- moved H2 20.3 mm to (22.9, 3.81)
- moved LOGO3 18.6 mm to (19.1, 4.32)
- moved C4 17.6 mm to (19.2, 3.11), turned to 270 degrees
- moved U$11 16.9 mm to (36.8, 22.3), turned to 90 degrees
- moved C3 14.7 mm to (17.3, 3.11), turned to 270 degrees
- moved U$17 11.1 mm to (21.0, 15.5), flipped to the bottom, turned to 270 degrees
- moved U$19 11.0 mm to (19.4, 16.3), flipped to the bottom, turned to 270 degrees
- moved C6 8.84 mm to (17.8, 13.7), turned to 90 degrees
- moved U$18 7.33 mm to (19.3, 11.9), flipped to the bottom, turned to 270 degrees
- moved C1 4.95 mm to (21.6, 14.1)
- moved FD2 4.84 mm to (40.6, 26.7)
- moved FD4 4.84 mm to (40.6, 26.7)
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Connections:
- removed net BLUE_P: J3.5, J7.5, VDD_A.2
- removed net GRN_P: HV_IN.1, J3.3, J6.1, J7.3
- removed net N$8: C5.2, L1.P$1, U2.5
- removed net VDD_A: S1.1, VDD_A.1
- removed net VREG_3V3: C6.1, C7.1, L1.P$2, S1.2, U2.1
- new net N$1: C9.1, U3.4
- new net N$6: R1.1, R2.2, U3.7
- new net N$9: C5.1, R3.2, U3.5
- new net SW: C9.2, L2.P$1, U3.12, U3.3
- new net VCC_1: BUCK_BP.2, J3.4, J7.4, PSEL.3, TP1.P$1, U1.10
- new net VCC_2: J3.3, J6.1, J7.3, PSEL.1
- net 3.3V: now also BUCK_BP.1, C10.1, C11.1, C14.1, L2.P$2, R1.2; no longer S1.3, U1.10
- net BLUE_N: now also J3.5, J7.5; no longer J3.4, J7.4
- net GND: now also C10.2, C11.2, C12.-, C14.2, C15.2, C5.2, C8.2, R2.1, U3.1, U3.11, U3.6; no longer C8.1, U2.4
- net N$7: now also R3.1, U3.8; no longer C5.1, U2.6
- net VREG_IN: now also C12.+, C15.1, C6.1, C7.1, C8.1, PSEL.2, U3.10, U3.2, U3.9; no longer C8.2, HV_IN.2, U2.2, U2.3
Routing:
- net VCC_1: track 0.00 -> 60.4 mm, vias 0 -> 2
- net VCC_2: track 0.00 -> 54.5 mm
- net GRN_P: track 36.2 -> 0.00 mm
- net VDD_A: track 27.7 -> 0.00 mm, vias 1 -> 0
- net BLUE_P: track 25.3 -> 0.00 mm
- net VREG_3V3: track 24.4 -> 0.00 mm, vias 2 -> 0
- net 3.3V: track 81.7 -> 61.4 mm, vias 3 -> 5
- net VREG_IN: track 23.7 -> 9.19 mm, vias 1 -> 4
- net SCL: track 57.7 -> 46.7 mm, vias 1 -> 2
- net N$9: track 0.00 -> 9.57 mm
- net GND: track 1.31 -> 8.52 mm, vias 29 -> 45
- net N$6: track 0.00 -> 5.44 mm
- net SW: track 0.00 -> 5.04 mm
- net N$7: track 2.14 -> 6.60 mm
- net SDA: track 71.4 -> 67.0 mm, vias 3 -> 5
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- added copper zone on layer 1, net 3.3V
- added copper zone on layer 1, net SW
- added copper zone on layer 16, net VREG_IN
- removed copper zone on layer 1, net N$8
- removed copper zone on layer 1, net VREG_3V3
Other:
- board size 48.3 x 27.9 mm -> 45.7 x 27.9 mm
- board text added: "v13"
- board text removed: "v12"

Commit message: post checklist changes
Parts:
- added U$5: (no value), output:#BP#0
- C10, C11: value 22UF -> 22uF
- L2: value 4.7μH -> 2.2uH; device SparkFun-Coils:INDUCTOR_4X4MM -> SparkFun-Coils:INDUCTOR_5X5MM
- moved LOGO3 22.3 mm to (6.99, 23.1)
- moved U$22 20.7 mm to (18.3, 5.65)
- moved R1 1.21 mm to (15.5, 8.32)
- moved C5 1.17 mm to (10.6, 8.32), turned to 180 degrees
- moved R2 1.17 mm to (17.3, 8.32)
- moved C9 1.08 mm to (8.45, 10.1), turned to 180 degrees
- moved U$19 1.08 mm to (19.4, 15.2)
- moved R3 1.04 mm to (19.1, 8.32)
- moved C15 1.02 mm to (9.53, 12.7)
- moved C6 1.02 mm to (17.8, 12.7)
- moved C7 1.02 mm to (7.62, 12.7)
- moved C8 1.02 mm to (15.9, 12.7)
- moved PSEL 1.02 mm to (19.3, 11.9)
- moved U$18 1.02 mm to (19.3, 10.9)
- moved U$30 1.02 mm to (18.2, 12.6)
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- renumbered BUCK_BP to BP
Routing:
- net SW: track 5.04 -> 6.66 mm
- net N$9: track 9.57 -> 10.6 mm
- net VREG_IN: track 9.19 -> 10.2 mm
- net VCC_2: track 54.5 -> 55.5 mm
- net N$1: track 3.91 -> 3.23 mm
- net 3.3V: track 61.4 -> 61.9 mm
- net GND: vias 45 -> 44
