File: Hardware/SparkFun_QwiicBus-Midpoint.brd (EAGLE design)
At the start: 45.7 x 27.9 mm, 88 parts, among them J1 QWIIC, J2 QWIIC, J3 RJ45, J7 RJ45, Q1 SI7120AD, U1 PCA9615, U3 LMR33630, U4 LTC4231 Hot Swap Controller

Commit message: pushing unsaved changes from double check
Parts:
- moved LOGO1 22.5 mm to (29.2, 19.1)
- moved U$15 17.6 mm to (12.7, 5.08), turned to 0 degrees
- moved U$24 0.72 mm to (21.1, 25.4), turned to 0 degrees
- moved R6 0.51 mm to (14.0, 7.75)
- moved U3 0.38 mm to (12.7, 11.6)
- moved L2 0.25 mm to (12.7, 17.1)
- moved C15 0.25 mm to (9.27, 12.7)
Routing:
- net N$12: track 11.1 -> 16.7 mm
- net SW: track 6.81 -> 9.07 mm
- net N$6: track 5.41 -> 4.69 mm
- net SDA: track 67.8 -> 68.5 mm
- net N$8: track 7.01 -> 7.52 mm
- net GND: vias 45 -> 46
- added copper zone on layer 15, net VREG_IN
- removed copper zone on layer 2, net VREG_IN
Other:
- board text added: "v14"
- board text removed: "v13"

Commit message: rolling back to non hot swap version
Parts:
- removed C13: 20nF, hotswap:0603
- removed C17: 39nF, hotswap:0805
- removed D1: SMAJ36A, hotswap:DO-214AC
- removed FRAME2: FRAME-LETTER, SparkFun-Aesthetics:CREATIVE_COMMONS
- removed Q1: SI7120AD, hotswap:1212-8
- removed R10: 23m, hotswap:2512
- removed R12: 10, SparkFun-Resistors:0603
- removed R13: 1k, SparkFun-Resistors:0603
- removed R14: 20k, SparkFun-Resistors:0603
- removed R15: 1M, SparkFun-Resistors:0603
- removed R4: 1.65K, hotswap:0603
- removed R5: 32.4k, hotswap:0603
- removed R6: 4.22k, hotswap:0603
- removed R9: 1020K, hotswap:0603
- removed U4: LTC4231 Hot Swap Controller, hotswap:QFN-12
- moved LOGO1 22.5 mm to (12.7, 3.81)
- moved U$15 12.5 mm to (12.2, 17.5)
- moved U$30 7.12 mm to (18.2, 12.6), turned to 0 degrees
- moved U$17 1.02 mm to (21.0, 14.6)
- moved PSEL 1.02 mm to (19.3, 11.9)
- moved C7 0.76 mm to (7.62, 12.7)
- moved U$18 0.76 mm to (19.3, 10.9)
- moved U$24 0.72 mm to (21.6, 24.9), turned to 270 degrees
- moved U$19 0.64 mm to (19.4, 15.2)
- moved C9 0.38 mm to (8.45, 10.1)
- moved U3 0.38 mm to (12.7, 11.9)
- moved C8 0.25 mm to (15.9, 12.7)
- moved L2 0.25 mm to (12.7, 17.3)
- moved C15 0.25 mm to (9.53, 12.7)
- moved C5 0.25 mm to (10.6, 8.32)
Connections:
- removed net N$10: R4.2, R9.1, U4.2
- removed net N$11: Q1.4, R12.2
- removed net N$12: Q1.5, Q1.6, Q1.7, Q1.8, Q1.PAD, R10.P$2, U4.11
- removed net N$16: R12.1, R13.2, U4.10
- removed net N$17: C13.1, R13.1
- removed net N$19: R14.1, U4.7
- removed net N$2: R5.1, U4.5
- removed net N$20: R15.1, U4.1
- removed net N$21: C17.1, U4.8
- removed net N$5: R5.2, R6.1, U4.4
- removed net N$8: R4.1, R6.2, U4.3
- removed net PWR_SRC: D1.C, PSEL.2, R10.P$1, R15.2, R9.2, U4.12
- net GND: no longer C13.2, C17.2, D1.A, U4.6, U4.EXP
- net VREG_IN: now also PSEL.2; no longer Q1.1, Q1.2, Q1.3, R14.2, U4.9
Routing:
- net 3.3V: track 37.6 -> 61.9 mm
- net VREG_IN: track 28.7 -> 10.2 mm, vias 3 -> 4
- net N$12: track 16.7 -> 0.00 mm
- net PWR_SRC: track 15.6 -> 0.00 mm
- net N$16: track 7.61 -> 0.00 mm
- net N$8: track 7.52 -> 0.00 mm
- net N$10: track 5.96 -> 0.00 mm
- net N$5: track 5.67 -> 0.00 mm
- net N$11: track 4.34 -> 0.00 mm
- net N$17: track 2.92 -> 0.00 mm
- net N$19: track 2.85 -> 0.00 mm
- net SW: track 9.07 -> 6.66 mm
- net N$2: track 2.35 -> 0.00 mm
- net N$20: track 2.25 -> 0.00 mm
- net N$21: track 2.15 -> 0.00 mm
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- added copper zone on layer 1, net 3.3V
- added copper zone on layer 16, net VREG_IN
- removed copper zone on layer 15, net 3.3V
- removed copper zone on layer 2, net GND
- removed copper zone on layer 15, net VREG_IN
Other:
- board text added: "v13"
- board text removed: "v14"
