File: Production/SparkFun_QwiicBus-Midpoint-Panel_v13b.brd (EAGLE design)
At the start: 198.1 x 119.4 mm, 574 parts, among them J1 QWIIC, J10 RJ45, J11 RJ45, J15 QWIIC, J16 QWIIC, J17 RJ45, J18 RJ45, J2 QWIIC, J22 QWIIC, J23 QWIIC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

Commit message: RE-panelization for stronger inner-support tabs
Other:
- board size 198.1 x 119.4 mm -> 228.9 x 134.6 mm
